File: 4.UI_controller/04.Hardware/02.UI_Control/UI_Control/_autosave-UI_Control.kicad_pcb (KiCad board)
At the start: 2 copper layers, 47 parts, among them J1 COM1, J2 USB_B_Mini, J3 LCD, J4 Conn_01x03_Male, J5 SWD, J6 12V, U1 STM32L412K8Tx, U2 TPS54202H, U3 MCP1812BT_033TT, U4 ST2378ETTR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

Commit message: update Layout
Parts:
- removed C13, C14: 100n, Capacitor_SMD:C_0603_1608Metric
- removed R10, R11, R12, R13, R14, R15, R16: 1.5k, Resistor_SMD:R_0603_1608Metric
- removed U4: ST2378ETTR, Package_SO:TSSOP-20_4.4x6.5mm_P0.65mm
- added Q1: Q_PMOS_DGS, Package_TO_SOT_SMD:SOT-23, F.Cu at (121.8, 48.9)
- C10, C9: value 10u -> 22u
- C3: value 10u -> 100n
- L1: value L -> 15uH
- R9: value 1.5k -> 100k; moved to F.Cu
- moved RV1 43.8 mm to (166.8, 43.7)
- moved U5 31.8 mm to (143.5, 48.3), turned to 270 degrees
- moved J6 22.2 mm to (118.0, 49.9)
- moved R9 20.7 mm to (121.6, 46.3)
- moved U1 16.9 mm to (130.3, 49.6), turned to 270 degrees
- moved J5 5.39 mm to (138.8, 58.6), turned to 0 degrees
- moved R8 5.04 mm to (132.3, 56.2), turned to 180 degrees
- moved J2 3.14 mm to (122.1, 60.1)
- moved C8 0.80 mm to (139.4, 53.9), turned to 180 degrees
Connections:
- C12 pad 2: GND -> Net-(C12-Pad2)
- J6 pad 1: +12V -> Net-(J6-Pad1)
- R6 pad 2: Net-(R6-Pad2) -> Net-(C12-Pad2)
- R7 pad 1: Net-(R6-Pad2) -> Net-(C12-Pad2)
- R9 pad 1: GND -> Net-(Q1-Pad2)
- R9 pad 2: /DB3_3V3 -> GND
- U1 pad 10: /DB5_3V3 -> (no net)
- U1 pad 11: /DB4_3V3 -> (no net)
- U1 pad 12: /DB3_3V3 -> (no net)
- U1 pad 13: /DB2_3V3 -> (no net)
- U1 pad 14: /DB1_3V3 -> (no net)
- U1 pad 15: /DB0_3V3 -> (no net)
- U1 pad 7: /DB7_3V3 -> (no net)
- U1 pad 8: /OE -> (no net)
- U1 pad 9: /DB6_3V3 -> (no net)
- U2 pad 4: Net-(R6-Pad2) -> Net-(C12-Pad2)
- U5 pad 10: (no net) -> /DB2
- U5 pad 11: (no net) -> /DB1
- U5 pad 12: (no net) -> /DB0
- U5 pad 4: (no net) -> /DB3
- U5 pad 5: (no net) -> /DB4
- U5 pad 6: (no net) -> /DB5
- U5 pad 7: (no net) -> /DB6
- U5 pad 9: (no net) -> /DB7
Routing:
- net /V0: track 47.3 -> 0.00 mm
- net /FS: track 41.8 -> 0.00 mm, vias 2 -> 0
- net /MD2: track 39.4 -> 0.00 mm, vias 2 -> 0
- net /RESET: track 35.4 -> 0.00 mm, vias 2 -> 0
- net /CD: track 28.9 -> 0.00 mm
- net /RD: track 26.6 -> 0.00 mm
- net /WR: track 21.0 -> 0.00 mm
- net /CE: track 20.8 -> 0.00 mm
- net +3V3: track 21.3 -> 4.40 mm
- net /DB3_3V3: track 15.2 -> 0.00 mm, vias 1 -> 0
- net /USB_D+: track 14.8 -> 0.00 mm
- net /DB4_3V3: track 13.9 -> 0.00 mm, vias 1 -> 0
- net /DB2_3V3: track 13.6 -> 0.00 mm, vias 1 -> 0
- net /USB_D-: track 12.7 -> 0.00 mm
- net /DB5_3V3: track 12.4 -> 0.00 mm, vias 1 -> 0
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