File: 4.UI_controller/04.Hardware/02.UI_Control/UI_Control/UI_Control.kicad_pcb (KiCad board)
At the start: 2 copper layers, 47 parts, among them J1 COM1, J2 USB_B_Mini, J3 LCD, J4 Conn_01x03_Male, J5 SWD, J6 12V, U1 STM32L412K8Tx, U2 TPS54202H, U3 MCP1812BT_033TT, U4 ST2378ETTR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

Commit message: update Layout
Parts:
- removed R13, R14, R15, R16: 1.5k, Resistor_SMD:R_0603_1608Metric
- removed RV1: R_POT_TRIM, Potentiometer_THT:Potentiometer_Vishay_T73YP_Vertical
- added H1: MountingHole, MountingHole:MountingHole_2.5mm, F.Cu at (183.0, 112.0)
- added H2: MountingHole, MountingHole:MountingHole_2.5mm, F.Cu at (131.5, 74.0)
- added H3: MountingHole, MountingHole:MountingHole_2.5mm, F.Cu at (130.2, 111.5)
- added J7: Conn_01x04_Male, Connector_Phoenix_MC:PhoenixContact_MC_1,5_4-G-3.81_1x04_P3.81mm_Horizontal, F.Cu at (138.5, 109.3)
- added Q1: Q_PMOS_DGS, Package_TO_SOT_SMD:SOT-23, F.Cu at (130.5, 80.9)
- added Q2: DMN6140L, Package_TO_SOT_SMD:SOT-23, F.Cu at (190.1, 87.3)
- C10, C9: value 10u -> 22u
- C3: value 10u -> 100n
- J1: footprint Connector_PinHeader_2.54mm:PinHeader_1x03_P2.54mm_Vertical -> Connector_Phoenix_MC:PhoenixContact_MC_1,5_3-G-3.81_1x03_P3.81mm_Horizontal
- J6: footprint Connector_PinHeader_2.54mm:PinHeader_1x02_P2.54mm_Vertical -> Connector_Phoenix_MC:PhoenixContact_MC_1,5_2-G-3.81_1x02_P3.81mm_Horizontal
- L1: value L -> 15uH
- R10: value 1.5k -> 6.8k; footprint Resistor_SMD:R_0603_1608Metric -> Resistor_SMD:R_1206_3216Metric; moved to F.Cu
- R11: value 1.5k -> 1.2k; footprint Resistor_SMD:R_0603_1608Metric -> Resistor_SMD:R_1206_3216Metric; moved to F.Cu
- R12: value 1.5k -> 100; footprint Resistor_SMD:R_0603_1608Metric -> Resistor_SMD:R_1206_3216Metric; moved to F.Cu
- R9: value 1.5k -> 100k; moved to F.Cu
- U4: value ST2378ETTR -> MCP4725A; footprint Package_SO:TSSOP-20_4.4x6.5mm_P0.65mm -> Package_TO_SOT_SMD:SOT-23-6
- U6: value MCP4541T -> OPA2990; footprint Package_SO:MSOP-8_3x3mm_P0.65mm -> Package_SO:TSSOP-8_4.4x3mm_P0.65mm
- moved C16 104.4 mm to (186.0, 78.0), turned to 180 degrees
- moved R5 103.1 mm to (186.6, 89.7), turned to 270 degrees
- moved R4 94.6 mm to (185.0, 89.7), turned to 270 degrees
- moved C14 91.9 mm to (181.1, 80.8)
- moved R1 89.0 mm to (163.6, 84.5), turned to 270 degrees
- moved R6 81.5 mm to (148.1, 80.8), turned to 90 degrees
- moved C2 77.5 mm to (163.6, 87.6), turned to 270 degrees
- moved R3 75.2 mm to (160.8, 92.0)
- moved R7 70.9 mm to (149.7, 80.8), turned to 90 degrees
- moved C13 70.7 mm to (161.5, 89.6), turned to 270 degrees
- moved C6 64.8 mm to (145.2, 81.0), turned to 180 degrees
- moved D1 64.7 mm to (138.1, 91.1), turned to 180 degrees
- moved L1 64.2 mm to (135.4, 82.3), turned to 90 degrees
- moved C4 63.2 mm to (141.1, 88.1), turned to 90 degrees
- moved R12 60.6 mm to (190.2, 90.5), turned to 180 degrees
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Connections:
- C11 pad 1: +3V3 -> GND
- C11 pad 2: GND -> +3V3
- C12 pad 2: GND -> Net-(C12-Pad2)
- C13 pad 1: GND -> +3V3
- C13 pad 2: +3V3 -> GND
- C14 pad 1: +5V -> GND
- C14 pad 2: GND -> +5V
- C16 pad 2: +3V3 -> /VEE
- C4 pad 1: +5VA -> +5V
- D1 pad 1: +5VA -> +5V
- D1 pad 2: +5V -> +5VA
- J4 pad 1: GND -> Net-(J4-Pad1)
- J4 pad 3: Net-(J4-Pad3) -> +3V3
- J6 pad 1: +12V -> Net-(J6-Pad1)
- R10 pad 1: GND -> /V0
- R10 pad 2: /DB4_3V3 -> Net-(R10-Pad2)
- R11 pad 1: GND -> Net-(R10-Pad2)
- R11 pad 2: /DB2_3V3 -> +5V
- R12 pad 1: GND -> /BACKLIGHT
- R12 pad 2: /DB5_3V3 -> Net-(Q2-Pad1)
- R6 pad 2: Net-(R6-Pad2) -> Net-(C12-Pad2)
- R7 pad 1: Net-(R6-Pad2) -> Net-(C12-Pad2)
- R9 pad 1: GND -> Net-(Q1-Pad2)
- R9 pad 2: /DB3_3V3 -> GND
- U1 pad 10: /DB5_3V3 -> /WR
- U1 pad 11: /DB4_3V3 -> /RESET
- U1 pad 12: /DB3_3V3 -> /RD
- U1 pad 13: /DB2_3V3 -> /CD
- U1 pad 14: /DB1_3V3 -> /MD2
- U1 pad 15: /DB0_3V3 -> /FS
- U1 pad 18: /CE -> (no net)
- U1 pad 2: /CD -> (no net)
- U1 pad 25: (no net) -> /BACKLIGHT
- U1 pad 26: /FS -> (no net)
- U1 pad 27: /MD2 -> /GPIO1
- U1 pad 28: /RESET -> /GPIO2
- U1 pad 3: /RD -> (no net)
- U1 pad 6: /WR -> (no net)
- U1 pad 7: /DB7_3V3 -> (no net)
- U1 pad 8: /OE -> (no net)
- U1 pad 9: /DB6_3V3 -> /CE
- U2 pad 4: Net-(R6-Pad2) -> Net-(C12-Pad2)
- U3 pad 2: +5VA -> +5V
- U4 pad 1: +3V3 -> Net-(U4-Pad1)
- U4 pad 2: /DB3_3V3 -> GND
- U4 pad 3: /DB4 -> +3V3
- U4 pad 4: /DB2_3V3 -> /SDA
- U4 pad 5: /DB5 -> /SCL
- U4 pad 6: /DB1_3V3 -> GND
- U5 pad 10: (no net) -> /DB5
- U5 pad 11: (no net) -> /DB6
- U5 pad 12: (no net) -> /DB7
- U5 pad 4: (no net) -> /DB0
- U5 pad 5: (no net) -> /DB1
- U5 pad 6: (no net) -> /DB2
- U5 pad 7: (no net) -> /DB3
- U5 pad 9: (no net) -> /DB4
- U6 pad 1: +3V3 -> /V0
- U6 pad 2: /SCL -> Net-(R10-Pad2)
- U6 pad 3: /SDA -> Net-(U4-Pad1)
- U6 pad 4: GND -> /VEE
- U6 pad 5: +3V3 -> GND
- U6 pad 6: Net-(J4-Pad3) -> Net-(U6-Pad6)
- U6 pad 7: GND -> Net-(U6-Pad6)
- U6 pad 8: +3V3 -> +5V
Routing:
- net +3V3: track 21.3 -> 171.3 mm, vias 0 -> 6
- net +5V: track 0.00 -> 119.8 mm, vias 0 -> 2
- net GND: track 34.8 -> 128.2 mm, vias 1 -> 12
- net /BACKLIGHT: track 0.00 -> 45.5 mm, vias 0 -> 2
- net /FS: track 41.8 -> 7.03 mm, vias 2 -> 0
- net /V0: track 47.3 -> 14.8 mm
- net /MD2: track 39.4 -> 7.12 mm, vias 2 -> 0
- net /GPIO1: track 0.00 -> 30.6 mm
- net /SDA: track 15.4 -> 45.2 mm, vias 0 -> 2
- net /VEE: track 8.74 -> 38.1 mm, vias 0 -> 2
- net /RESET: track 35.4 -> 6.27 mm, vias 2 -> 0
- net /GPIO2: track 0.00 -> 29.0 mm
- net /USART_TX: track 0.00 -> 22.3 mm
- net /SCL: track 21.8 -> 43.9 mm, vias 0 -> 2
- net +12V: track 0.00 -> 21.3 mm
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- added copper zone on B.Cu, net GND
- added copper zone on F.Cu, net GND
Other:
- board outline added: 81.5 x 45.5 mm
